File: PCB_rev_B4/Replicape_B4.sch (EAGLE design)
At the start: 257 parts, among them IC1 TMC2100-LA, IC10 74AHC1G126DCK, IC11 74AHC1G126DCK, IC12 TMC2100-LA, IC13 74AHC1G126DCK, IC14 74AHC1G126DCK, IC15 TMC2100-LA, IC16 74AHC1G126DCK, IC17 74AHC1G126DCK, IC18 74AHC1G126DCK, IC19 74AHC1G126DCK, IC2 TMC2100-LA, IC20 74AHC1G126DCK, IC21 74AHC1G126DCK, IC22 74AHC1G126DCK, IC3 74AHC1G126DCK, IC4 74AHC1G126DCK, IC5 TMC2100-LA, IC6 74AHC1G126DCK, IC7 74AHC1G126DCK, IC8 74AHC1G126DCK, IC9 74AHC1G126DCK, P8 F-2X23-, P9 F-2X23-, Q1 AON6758, Q2 AON6758, Q3 AON6758, U1 SN74AHC595PW, U10 RT8268, U11 PCA9685PW, U18 CAT24C256, U19 CD4050BD, U2 SN74AHC595PW, U3 SN74AHC595PW, U4 SN74AHC595PW, U5 SN74AHC595PW, U6 RT8268, U8 FI-RE41S-HFRIGHT_ANGLE, X1 22-05-7038-03, X10 22-05-7038-03, X11 22-05-7028-02, X12 22-05-7048-04, X13 22-05-7038-03, X15 22-05-7048-04, X16 22-05-7048-04, X18 22-05-7048-04, X19 22-05-7038-03, X2 MSTBA4, X20 MSTBA4, X21 MSTBA2, X22 22-05-7038-03, X23 22-05-7038-03, X3 MSTBA2, X4 22-05-7048-04, X5 22-05-7028-02, X6 22-05-7028-02, X7 22-05-7028-02, X8 22-05-7028-02, X9 22-05-7048-04

Commit message: changed the b4 version from 4 layer to 2 layer pcb and removed drc failures
Parts:
- removed C94, C95, C96, C97, C98: 100uF, Panasonic-EEEFK_EEEFP:C
- removed LED0, LED8: blue, led:LEDCHIP-LED0603
- removed Q6, Q7: (no value), semicon-smd-ipc:NPN-TRANSISTOR_SOT23
- removed R65, R66: 4.7K, rcl:R-EU_R0402
- removed R70, R71: 2.2R, rcl:R-EU_R0402
- removed U11: PCA9685PW, custom:PCA9685PW
- removed U18: CAT24C256, custom:CAT24C256
- removed U19: CD4050BD, TI-CD4050BD:CD4050BD
- removed X18: 22-05-7048-04, con-molex:22-05-7048-04
- removed X19, X22, X23: 22-05-7038-03, con-molex:22-05-7038-03
- removed X20: MSTBA4, con-phoenix-508:MSTBA4
- removed X21: MSTBA2, con-phoenix-508:MSTBA2
- added C11: 10uF, rcl:C-EUC1206
- added C16: 10nF, rcl:C-EUC0402
- added C24, C34: 0.1uF, rcl:C-EUC0402
- added C60: 4.7uF, rcl:C-EUC0402
- added J500, J501, J502, J503, J504: 22-05-7048-04, con-molex:22-05-7048-04
- added U7, U9: SN74AHC595PW, sn74hc595:SN74AHC595PW
- added X14: MSTBA4, con-phoenix-508:MSTBA4
- C1, C9: value 22nF -> 10uF; device rcl:C-EUC0402 -> rcl:C-EUC1206; MPN C1005X7R1E223K050BB -> CL31B106KAHNNNE
- C10, C13, C2: value 0.1uF -> 10uF; device rcl:C-EUC0402 -> rcl:C-EUC1206; MPN CL10B104KB8NNND -> CL31B106KAHNNNE
- C12, C18, C25, C26, C46, C62, C65, C68, C75, C76, C77, C78: value 4.7uF -> 0.1uF; MPN GRM155R60J475ME47D -> CL10B104KB8NNND
- C14, C17: value 0.1uF -> 1nF; MPN CL10B104KB8NNND -> C1005X7R1H102K050BA
- C15, C20: value 0.1uF -> 10nF; MPN CL10B104KB8NNND -> CL05B103KB5NNNC
- C21: value 4.7uF -> 10nF; MPN GRM155R60J475ME47D -> CL05B103KB5NNNC
- C3: value 22nF -> 4.7nF; MPN C1005X7R1E223K050BB -> CL05B472KA5NNNC
- C32, C63: value 0.1uF -> 4.7nF; MPN CL10B104KB8NNND -> CL05B472KA5NNNC
- C33, C45: value 4.7uF -> 22nF; MPN GRM155R60J475ME47D -> C1005X7R1E223K050BB
- C35, C4, C41, C42, C43, C5, C6, C61: value 0.1uF -> 4.7uF; MPN CL10B104KB8NNND -> GRM155R60J475ME47D
- C47, C48, C53: value 10uF -> 4.7uF; device rcl:C-EUC1206 -> rcl:C-EUC0402; MPN CL31B106KAHNNNE -> GRM155R60J475ME47D
- C49, C54, C55: value 10nF -> 4.7uF; MPN CL05B103KB5NNNC -> GRM155R60J475ME47D
- C50: value 10nF -> 0.1uF; MPN CL05B103KB5NNNC -> CL10B104KB8NNND
- C51: value 1nF -> 22nF; MPN C1005X7R1H102K050BA -> C1005X7R1E223K050BB
- C52: value 10uF -> 0.1uF; device rcl:C-EUC1206 -> rcl:C-EUC0402; MPN CL31B106KAHNNNE -> CL10B104KB8NNND
- C56: value 1nF -> 0.1uF; MPN C1005X7R1H102K050BA -> CL10B104KB8NNND
- C57: value 4.7nF -> 22nF; MPN CL05B472KA5NNNC -> C1005X7R1E223K050BB
- C58: value 4.7nF -> 0.1uF; MPN CL05B472KA5NNNC -> CL10B104KB8NNND
- C59: value 4.7nF -> 4.7uF; MPN CL05B472KA5NNNC -> GRM155R60J475ME47D
- C7: value 22nF -> 0.1uF; MPN C1005X7R1E223K050BB -> CL10B104KB8NNND
- C79: value 4.7uF -> 100uF; device rcl:C-EUC0402 -> Panasonic-EEEFK_EEEFP:C; MPN GRM155R60J475ME47D -> RHS1V101MCN1GS
- C80, C81: value 10uF -> 100uF; device rcl:C-EUC1206 -> Panasonic-EEEFK_EEEFP:C; MPN CL31B106KAHNNNE -> RHS1V101MCN1GS
- C82, C83: value 0.1uF -> 100uF; device rcl:C-EUC0402 -> Panasonic-EEEFK_EEEFP:C; MPN CL10B104KB8NNND -> RHS1V101MCN1GS
- IC1, IC12, IC15, IC2, IC5: value TMC2100-LA -> 74AHC1G126DCK; device we-chip:TMC2100-LA -> 74xx-little-de:74AHC1G126DCK; MPN TMC2100-LA-T -> M74VHC1GT126DF1G
- IC18, IC19, IC20, IC21, IC22: value 74AHC1G126DCK -> TMC2100-LA; device 74xx-little-de:74AHC1G126DCK -> we-chip:TMC2100-LA; MPN M74VHC1GT126DF1G -> TMC2100-LA-T
- R1, R2, R3, R30, R4, R7, R8: value 0.1R -> 4.7K; device rcl:R-EU_R0805 -> rcl:R-EU_R0402; MPN RL1220S-R10-F -> RC0402JR-074K7L
- R10, R29: value 0.1R -> 10K; device rcl:R-EU_R0805 -> rcl:R-EU_R0402; MPN RL1220S-R10-F -> RC0402FR-0710KL
- R11, R14, R28, R32, R33, R36, R45: value 4.7K -> 10K; MPN RC0402JR-074K7L -> RC0402FR-0710KL
- R12: value 44.3K,1% -> 4K7, 1%; MPN RC1005F4422CS -> RC0402FR-074K7L
- R16: value 4.7K -> 10K,1%; MPN RC0402JR-074K7L -> RC0402FR-0710KL
- R17: value 4K7, 1% -> 44.3K,1%; MPN RC0402FR-074K7L -> RC1005F4422CS
- R18: value 4K7, 1% -> 10K,1%; MPN RC0402FR-074K7L -> RC0402FR-0710KL
- R19: value 4.7K -> 120K,1%; MPN RC0402JR-074K7L -> RMCF0402FT120K
- R20, R23: value 4.7K -> 39K; MPN RC0402JR-074K7L -> RC1005J393CS
- R22: value 10K,1% -> 4.7K; MPN RC0402FR-0710KL -> RC0402JR-074K7L
- R26: value 39K -> 4.7K; MPN RC1005J393CS -> RC0402JR-074K7L
- R27, R31, R35, R39: value 10K -> 2.2R; MPN RC0402FR-0710KL -> RC1005J2R2CS
- R38, R58, R6, R60: value 10K -> 4.7K; MPN RC0402FR-0710KL -> RC0402JR-074K7L
- R42: value 120K,1% -> 4.7K; MPN RMCF0402FT120K -> RC0402JR-074K7L
- R43: value 10K,1% -> 2.2R; MPN RC0402FR-0710KL -> RC1005J2R2CS
- R44: value 39K -> 10K; MPN RC1005J393CS -> RC0402FR-0710KL
- R48, R51, R54, R55, R56, R57: value 4.7K -> 0.1R; device rcl:R-EU_R0402 -> rcl:R-EU_R0805; MPN RC0402JR-074K7L -> RL1220S-R10-F
- R49, R50: value 10K -> 0.1R; device rcl:R-EU_R0402 -> rcl:R-EU_R0805; MPN RC0402FR-0710KL -> RL1220S-R10-F
- R52, R53: value 2.2R -> 0.1R; device rcl:R-EU_R0402 -> rcl:R-EU_R0805; MPN RC1005J2R2CS -> RL1220S-R10-F
- R59: value 2.2R -> 4.7K; MPN RC1005J2R2CS -> RC0402JR-074K7L
- R9: value 0.1R -> 4K7, 1%; device rcl:R-EU_R0805 -> rcl:R-EU_R0402; MPN RL1220S-R10-F -> RC0402FR-074K7L
- U1: value SN74AHC595PW -> PCA9685PW; device sn74hc595:SN74AHC595PW -> custom:PCA9685PW; MPN MC74HC595ADTR2G -> PCA9685PW,112
- U10, U6: value RT8268 -> SN74AHC595PW; device SparkFun:RT8268 -> sn74hc595:SN74AHC595PW; MPN RT8268GFP -> MC74HC595ADTR2G
- U2: value SN74AHC595PW -> CAT24C256; device sn74hc595:SN74AHC595PW -> custom:CAT24C256; MPN MC74HC595ADTR2G -> CAT24C256WI-GT3
- U3: value SN74AHC595PW -> CD4050BD; device sn74hc595:SN74AHC595PW -> TI-CD4050BD:CD4050BD; MPN MC74HC595ADTR2G -> CD4050BDR
- U4, U5: value SN74AHC595PW -> RT8268; device sn74hc595:SN74AHC595PW -> SparkFun:RT8268; MPN MC74HC595ADTR2G -> RT8268GFP
- U8: value FI-RE41S-HFRIGHT_ANGLE -> SN74AHC595PW; device JAE_By_element14_Batch_1:FI-RE41S-HFRIGHT_ANGLE -> sn74hc595:SN74AHC595PW; MPN (none) -> MC74HC595ADTR2G
- X10: value 22-05-7038-03 -> 22-05-7048-04; device con-molex:22-05-7038-03 -> con-molex:22-05-7048-04; MPN 640455-3 -> 640455-4
- X11: value 22-05-7028-02 -> MSTBA2; device con-molex:22-05-7028-02 -> con-phoenix-508:MSTBA2; MPN 640455-2 -> 39532-1002
- X12: value 22-05-7048-04 -> MSTBA4; device con-molex:22-05-7048-04 -> con-phoenix-508:MSTBA4; MPN 640455-4 -> 39532-1004
- X13: value 22-05-7038-03 -> MSTBA2; device con-molex:22-05-7038-03 -> con-phoenix-508:MSTBA2; MPN 640455-3 -> 39532-1002
- X15, X16, X4: value 22-05-7048-04 -> 22-05-7028-02; device con-molex:22-05-7048-04 -> con-molex:22-05-7028-02; MPN 640455-4 -> 640455-2
- X2: value MSTBA4 -> 22-05-7028-02; device con-phoenix-508:MSTBA4 -> con-molex:22-05-7028-02; MPN 39532-1004 -> 640455-2
- X3: value MSTBA2 -> 22-05-7028-02; device con-phoenix-508:MSTBA2 -> con-molex:22-05-7028-02; MPN 39532-1002 -> 640455-2
- X5, X6, X7, X8: value 22-05-7028-02 -> 22-05-7038-03; device con-molex:22-05-7028-02 -> con-molex:22-05-7038-03; MPN 640455-2 -> 640455-3
- X9: value 22-05-7048-04 -> 22-05-7038-03; device con-molex:22-05-7048-04 -> con-molex:22-05-7038-03; MPN 640455-4 -> 640455-3
- XC1: value MSTBA4-CONNECTOR -> MSTBV2-CONNECTOR; device con-phoenix-508:MSTBA4-CONNECTOR -> con-phoenix-508:MSTBV2-CONNECTOR; MPN 39530-0004 -> 39530-0002
- XC4: value MSTBV2-CONNECTOR -> MSTBA4-CONNECTOR; device con-phoenix-508:MSTBV2-CONNECTOR -> con-phoenix-508:MSTBA4-CONNECTOR; MPN 39530-0002 -> 39530-0004
- renumbered P8 to P2, P9 to P1, SV2 to SV1, U$4 to U$1
Connections:
- removed net AUX_0: U8.10, U8.11
- removed net A_A1: U8.22
- removed net A_A2: U8.21
- removed net A_B1: U8.20
- removed net A_B2: U8.19
- removed net FAN0: Q6.B, R34.2, U11.LED7
- removed net FAN0_OUT: LED0.C, Q6.C, U8.14
- removed net FAN1: Q7.B, R33.2, U11.LED8
- removed net FAN1_OUT: LED5.C, Q7.C, U8.15
- removed net IREF_E: C79.1, R35.2, R60.1
- removed net IREF_H: C75.1, R31.1, R50.2
- removed net IREF_X: C77.1, R41.1, R49.2
- removed net IREF_Y: C76.1, R37.1, R6.2
- removed net IREF_Z: C78.1, R27.2, R58.1
- removed net N$21: LED0.A, R25.1
- removed net N$33: C22.1, IC1.VCP
- removed net N$34: IC3A.I, U1.QE
- removed net N$47: C33.2, IC2.5VOUT, R59.1
- removed net N$48: C35.1, IC2.VCP
- removed net N$55: IC5.SDO_NAO_CFG0, U3.QD
- removed net N$56: IC2.ENCB_DCEN_CFG4, U2.QC
- removed net N$70: C39.2, IC12.CPO
- removed net N$71: IC12.BRB, R29.2
- removed net N$9: LED5.A, R19.1
- removed net X_CFG1: IC1.SDI_NAI_CFG1, IC4A.O
- removed net X_CFG2: IC1.SCK_CFG2, IC3A.O
- new net IREF_Z10: C61.1, R44.2, R45.1
- new net IREF_Z6: C49.1, R36.2, R37.1
- new net IREF_Z7: C55.1, R40.2, R41.1
- new net IREF_Z8: C37.1, R28.2, R29.1
- new net IREF_Z9: C43.1, R32.2, R33.1
- new net N$122: IC20.OB2, J502-4.S
- new net N$123: IC20.OA1, J502-2.S
- new net N$138: IC20.OA2, J502-1.S
- new net N$139: IC20.OB1, J502-3.S
- new net N$167: IC12A.I, U10.QG
- new net N$168: IC17A.I, U10.QE
- new net N$180: IC17A.OE, U10.QF
- new net N$181: C58.1, IC22.VCC, R43.2
- new net N$224: IC22.OA2, J500-1.S
- new net N$225: IC22.OB1, J500-3.S
- net +3V3: now also C19.1, C22.1, C24.1, C25.1, C26.1, C27.1, C28.1, C29.1, C31.1, C38.1, C50.1, C56.1, C62.1, C7.1, IC12P.VCC, IC15P.VCC, IC18.VCC_IO, IC19.VCC_IO, IC20.VCC_IO, IC21.VCC_IO, IC22.VCC_IO, IC5P.VCC, IC6P.VCC, IC7P.VCC, R22.2, R30.2, R34.2, R38.2, R42.2, R46.2, U10.VCC, U10.~SRCLR, U2.A2, U6.VCC, U6.~SRCLR, U7.VCC, U7.~SRCLR, U8.VCC, U8.~SRCLR, U9.VCC, U9.~SRCLR, X1-1.S; no longer C13.1, C14.1, C15.1, C2.1, C41.1, C42.1, C5.1, C61.1, C63.1, C84.1, C85.1, C86.1, C87.1, C88.1, IC1.VCC_IO, IC12.VCC_IO, IC15.VCC_IO, IC18P.VCC, IC19P.VCC, IC2.VCC_IO, IC20P.VCC, IC21P.VCC, IC22P.VCC, IC5.VCC_IO, R23.2, R24.2, R28.2, R36.2, R51.2, R54.2, U1.VCC, U1.~SRCLR, U18.A2, U18.VCC, U19.VCC, U2.~SRCLR, U3.~SRCLR, U4.VCC, U4.~SRCLR, U5.VCC, U5.~SRCLR, X23-1.S
- net DALLAS_W1: now also X1-2.S; no longer X23-2.S
- net DIR_E: now also IC21.REFR_DIR; no longer IC12.REFR_DIR
- net DIR_H: now also IC22.REFR_DIR; no longer IC15.REFR_DIR
- net DIR_X: now also IC18.REFR_DIR; no longer IC1.REFR_DIR
- net DIR_Y: now also IC19.REFR_DIR; no longer IC2.REFR_DIR
- net DIR_Z: now also IC20.REFR_DIR; no longer IC5.REFR_DIR
- net ENABLE: now also R22.1, U1.~OE; no longer R23.1, U11.~OE
- net ENABLE_E: now also IC21.DRV_ENN_CFG6, IC6A.O; no longer IC12.DRV_ENN_CFG6, IC19A.O
- net ENABLE_H: now also IC22.DRV_ENN_CFG6, IC7A.O; no longer IC15.DRV_ENN_CFG6, IC22A.O
- net ENABLE_X: now also IC18.DRV_ENN_CFG6, IC3A.O; no longer IC1.DRV_ENN_CFG6, IC18A.O
- net ENABLE_Y: now also IC19.DRV_ENN_CFG6, IC4A.O; no longer IC2.DRV_ENN_CFG6, IC20A.O
- net ENABLE_Z: now also IC20.DRV_ENN_CFG6, IC5A.O; no longer IC21A.O, IC5.DRV_ENN_CFG6
- net END_STOP_X_1: now also U3.G=A; no longer U19.G=A
- net END_STOP_X_1_IN: now also R1.1, U3.A, X5-1.S; no longer R61.1, U19.A, U8.4, X22-1.S
- net END_STOP_X_2: now also U3.J=D; no longer U19.J=D
- net END_STOP_X_2_IN: now also IC2A.O, R4.1, U3.D, X8-1.S; no longer IC6A.O, R64.1, U19.D, X10-1.S
- net END_STOP_Y_1: now also U3.H=B; no longer U19.H=B
- net END_STOP_Y_1_IN: now also R2.1, U3.B, X6-1.S; no longer R62.1, U19.B, X1-1.S
- net END_STOP_Y_2: now also U3.K=E; no longer U19.K=E
- net END_STOP_Y_2_IN: now also IC1A.O, R5.1, U3.E, X9-1.S; no longer IC7A.O, R65.1, U19.E, X19-1.S
- net END_STOP_Z_1: now also U3.I=C; no longer U19.I=C
- net END_STOP_Z_1_IN: now also R3.1, U3.C, X7-1.S; no longer R63.1, U19.C, X13-1.S
- net END_STOP_Z_2: now also U3.L=F; no longer U19.L=F
- net END_STOP_Z_2_IN: now also R6.1, U3.F, X10-1.S; no longer R66.1, U19.F, U8.13, X12-1.S
- net EN_EH: now also IC6A.I, IC7A.I, U9.QA; no longer IC19A.I, IC22A.I, U4.QA
- net EN_XYZ: now also IC3A.I, IC4A.I, IC5A.I, U6.QA; no longer IC18A.I, IC20A.I, IC21A.I, U1.QA
- net E_A1: now also IC21.OA1, J501-2.S; no longer IC12.OA1, U8.27, X9-1.S
- net E_A2: now also IC21.OA2, J501-1.S; no longer IC12.OA2, U8.26, X9-2.S
- net E_B1: now also IC21.OB1, J501-3.S; no longer IC12.OB1, U8.25, X9-3.S
- net E_B2: now also IC21.OB2, J501-4.S; no longer IC12.OB2, U8.24, X9-4.S
- net FAN2: now also R61.2, U1.LED9; no longer R32.2, U11.LED9
- net FAN3: now also R60.2, U1.LED10; no longer R5.2, U11.LED10
- net FAULT_E: now also IC21.SWN_DIAG0, R42.1; no longer IC12.SWN_DIAG0, R36.1
- net FAULT_H: now also IC22.SWN_DIAG0, R46.1; no longer IC15.SWN_DIAG0, R51.1
- net FAULT_X: now also IC18.SWN_DIAG0, R30.1; no longer IC1.SWN_DIAG0, R54.1
- net FAULT_Y: now also IC19.SWN_DIAG0, R34.1; no longer IC2.SWN_DIAG0, R24.1
- net FAULT_Z: now also IC20.SWN_DIAG0, R38.1; no longer IC5.SWN_DIAG0, R28.1
- net GND: now also C1.2, C11.2, C20.2, C22.2, C24.2, C28.2, C3.2, C32.2, C34.2, C35.1, C37.2, C38.2, C41.1, C47.1, C50.2, C53.1, C55.2, C56.2, C59.1, C60.2, C69.1, C7.2, C71.1, C73.1, C79.-, C80.-, C81.-, C82.-, C83.-, C9.2, D2.A, IC12P.GND, IC15P.GND, IC18.CLK, IC18.GND, IC18.GNDA, IC18.SPI_MODE, IC18.TST_MODE, IC19.CLK, IC19.GND, IC19.GNDA, IC19.SPI_MODE, IC19.TST_MODE, IC1P.GND, IC20.CLK, IC20.GND, IC20.GNDA, IC20.SPI_MODE, IC20.TST_MODE, IC21.CLK, IC21.GND, IC21.GNDA, IC21.SPI_MODE, IC21.TST_MODE, IC22.CLK, IC22.GND, IC22.GNDA, IC22.SPI_MODE, IC22.TST_MODE, IC2P.GND, IC5P.GND, LED2.C, R16.2, R18.2, R20.2, R21.1, R23.2, R49.1, R50.1, R51.1, R52.1, R53.1, R54.1, R55.1, R56.1, R57.1, R60.1, R61.1, U1.VSS, U10.~OE, U2.A0, U2.A1, U3.VSS, U4.EP, U5.EP, U6.~OE, U7.GND, U7.~OE, U8.GND, U8.~OE, U9.GND, U9.~OE, X1-3.S, X14-1.1, X14-2.1, X2-1.S, X3-1.S, X4-1.S, X5-2.S, X6-2.S, X7-2.S, X8-2.S, X9-2.S; no longer C14.2, C17.2, C20.1, C21.1, C28.1, C32.1, C33.1, C37.1, C41.2, C45.2, C47.2, C53.2, C57.2, C59.2, C64.1, C68.1, C70.2, C71.2, C72.2, C73.2, C79.2, C80.2, C81.2, C82.2, C83.2, C94.-, C95.-, C96.-, C97.-, C98.-, D5.A, IC1.CLK, IC1.GND, IC1.GNDA, IC1.SPI_MODE, IC1.TST_MODE, IC12.CLK, IC12.GND, IC12.GNDA, IC12.SPI_MODE, IC12.TST_MODE, IC15.CLK, IC15.GND, IC15.GNDA, IC15.SPI_MODE, IC15.TST_MODE, IC18P.GND, IC19P.GND, IC2.CLK, IC2.GND, IC2.GNDA, IC2.SPI_MODE, IC2.TST_MODE, IC20P.GND, IC21P.GND, IC22P.GND, IC5.CLK, IC5.GND, IC5.GNDA, IC5.SPI_MODE, IC5.TST_MODE, LED4.C, Q6.E, Q7.E, R1.1, R10.1, R2.1, R22.2, R26.2, R29.1, R3.1, R30.1, R32.1, R33.1, R34.1, R4.1, R43.2, R44.2, R46.1, R5.1, R8.1, R9.1, U1.GND, U1.~OE, U10.EP, U11.VSS, U18.A0, U18.A1, U18.GND, U19.VSS, U2.~OE, U3.GND, U3.~OE, U4.~OE, U5.~OE, U6.EP, U8.18, U8.23, U8.3, U8.30, U8.41, U8.9, X1-2.S, X11-1.S, X12-2.S, X13-2.S, X19-2.S, X2-1.1, X2-2.1, X22-2.S, X23-3.S, X7-1.S, X8-1.S
- net HEATER_E: now also U1.LED5; no longer U11.LED5
- net HEATER_E_OUT: now also C63.1, D5.A, LED4.C, R58.1, X13-2.1; no longer C59.1, D1.A, LED3.C, R55.1, U8.31, U8.32, U8.33, U8.34, U8.35, X3-2.1
- net HEATER_H: now also Q1.G, R7.2, U1.LED3; no longer Q2.G, R48.2, U11.LED3
- net HEATER_HBP: now also Q2.G, R21.2, U1.LED4; no longer Q1.G, R46.2, U11.LED4
- net I2C2_SCL: now also U1.SCL, U2.SCL; no longer U11.SCL, U18.SCL
- net I2C2_SDA: now also U1.SDA, U2.SDA; no longer U11.SDA, U18.SDA
- net IREF_E_RAW: now also R41.2, U1.LED14; no longer R60.2, U11.LED14
- net IREF_H_RAW: now also R45.2, U1.LED15; no longer R31.2, U11.LED15
- net IREF_X_RAW: now also R29.2, U1.LED11; no longer R41.2, U11.LED11
- net IREF_Y_RAW: now also R33.2, U1.LED12; no longer R37.2, U11.LED12
- net IREF_Z_RAW: now also R37.2, U1.LED13; no longer R58.2, U11.LED13
- net N$1: now also U1.LED0; no longer U11.LED0
- net N$100: now also IC22.BRB, R57.2; no longer IC15.SDO_NAO_CFG0, U5.QD
- net N$101: now also IC22.BRA, R56.2; no longer IC15.ENCB_DCEN_CFG4, U5.QC
- net N$102: now also C60.1, IC22.AIN_IREF, R44.1; no longer IC15.ENCA_DCIN_CFG5, U5.QB
- net N$103: now also C57.1, IC22.CPI; no longer IC17A.OE, U5.QH
- net N$104: now also IC17A.O, IC22.SCK_CFG2; no longer IC17A.I, U5.QG
- net N$105: now also IC22.OB2, J500-4.S; no longer IC16A.OE, U5.QF
- net N$106: now also IC22.OA1, J500-2.S; no longer IC16A.I, U5.QE
- net N$107: now also C59.2, IC22.5VOUT, R43.1; no longer C70.1, IC15.VCC, R52.2
- net N$108: now also C72.1, IC22.VCP; no longer C71.1, IC1.VCC, R53.2
- net N$109: now also IC12A.O, IC22.SDI_NAI_CFG1; no longer C73.1, IC5.VCC, R70.2
- net N$110: now also IC22.SDO_NAO_CFG0, U10.QD; no longer C72.1, IC2.VCC, R59.2
- net N$111: now also IC22.ENCB_DCEN_CFG4, U10.QC; no longer C74.1, IC12.VCC, R71.2
- net N$113: now also IC22.ENCA_DCIN_CFG5, U10.QB; no longer IC15.OB1, X18-3.S
- net N$114: now also LED6.C, X16-2.S; no longer LED7.C, X6-2.S
- net N$115: now also LED5.C, X15-2.S; no longer LED6.C, X5-2.S
- net N$117: now also LED5.A, R62.1; no longer LED6.A, R20.1
- net N$118: now also LED6.A, R63.1; no longer LED7.A, R21.1
- net N$119: now also IC12A.OE, U10.QH; no longer IC15.OA2, X18-1.S
- net N$12: now also IC15A.O, IC20.SCK_CFG2; no longer C9.2, IC15.CPO
- net N$120: now also U1.LED2; no longer U11.LED2
- net N$121: now also U1.LED1; no longer U11.LED1
- net N$127: now also LED4.A, R59.1; no longer LED3.A, R15.1
- net N$129: now also R15.1; no longer R14.1
- net N$13: now also C47.2, IC20.5VOUT, R35.1; no longer IC15.BRB, R9.2
- net N$130: now also LED3.A, R26.1; no longer LED2.A, R16.1
- net N$14: now also C68.1, IC20.VCP; no longer C7.2, IC5.CPO
- net N$15: now also IC10A.O, IC20.SDI_NAI_CFG1; no longer IC5.BRB, R7.2
- net N$16: now also IC20.SDO_NAO_CFG0, U8.QD; no longer C1.1, IC1.CPI
- net N$17: now also IC20.ENCB_DCEN_CFG4, U8.QC; no longer C1.2, IC1.CPO
- net N$18: now also IC20.ENCA_DCIN_CFG5, U8.QB; no longer IC1.BRB, R1.2
- net N$19: now also IC10A.OE, U8.QH; no longer IC1.BRA, R2.2
- net N$2: now also C45.2, IC20.CPO; no longer IC2.OB1, X15-3.S
- net N$20: now also IC10A.I, U8.QG; no longer C12.1, IC1.AIN_IREF, R49.1
- net N$22: now also IC15A.I, U8.QE; no longer IC2.OA2, X15-1.S
- net N$23: now also R16.1, R17.2, U4.FB; no longer R12.2, R22.1, U6.FB
- net N$233: now also R18.1, R19.2, U5.FB; no longer R42.2, R43.1, U10.FB
- net N$238: now also C21.2, L1.P$2, U5.SW; no longer C55.2, L2.P$2, U10.SW
- net N$24: now also IC15A.OE, U8.QF; no longer IC5.BRA, R8.2
- net N$240: now also R13.1, R14.1, X4-2.S; no longer R18.1, R40.1, X11-2.S
- net N$241: now also R11.1, R12.1, X3-2.S; no longer R17.1, R39.1, X7-2.S
- net N$242: now also C32.1, D3.A, LED3.C, Q2.D, R25.1, X12-3.1, X12-4.1; no longer C58.1, D2.A, LED2.C, Q1.D, R56.1, X20-3.1, X20-4.1
- net N$243: now also C20.1, U5.SS; no longer C54.1, U10.SS
- net N$244: now also C17.1, U5.COMP; no longer C56.1, U10.COMP
- net N$245: now also C21.1, U5.BOOT; no longer C55.1, U10.BOOT
- net N$246: now also C17.2, R23.1; no longer C56.2, R44.1
- net N$25: now also C16.2, D2.C, L2.P$2, U4.SW; no longer C50.2, D6.C, L1.P$2, U6.SW
- net N$26: now also C46.1, IC20.VCC, R35.2; no longer C25.1, IC5.AIN_IREF, R27.1
- net N$27: now also C51.2, IC21.CPO; no longer C7.1, IC5.CPI
- net N$28: now also IC21.BRB, R55.2; no longer IC10A.O, IC5.SCK_CFG2
- net N$29: now also IC21.BRA, R54.2; no longer IC5.OB2, X16-4.S
- net N$3: now also IC20.BRB, R53.2; no longer C3.2, IC2.CPO
- net N$30: now also C54.1, IC21.AIN_IREF, R40.1; no longer IC15.BRA, R10.2
- net N$31: now also C51.1, IC21.CPI; no longer C21.2, IC1.5VOUT, R53.1
- net N$32: now also IC16A.O, IC21.SCK_CFG2; no longer IC5.OA2, X16-1.S
- net N$35: now also C53.2, IC21.5VOUT, R39.1; no longer IC2.BRB, R3.2
- net N$36: now also C70.1, IC21.VCP; no longer IC2.BRA, R4.2
- net N$37: now also IC11A.O, IC21.SDI_NAI_CFG1; no longer IC5.OB1, X16-3.S
- net N$38: now also IC21.SDO_NAO_CFG0, U9.QD; no longer C18.1, IC2.AIN_IREF, R6.1
- net N$4: now also IC20.BRA, R52.2; no longer IC4A.OE, U1.QH
- net N$40: now also IC21.ENCB_DCEN_CFG4, U9.QC; no longer IC3A.OE, U1.QF
- net N$41: now also IC21.ENCA_DCIN_CFG5, U9.QB; no longer C3.1, IC2.CPI
- net N$42: now also IC11A.OE, U9.QH; no longer IC2.SCK_CFG2, IC8A.O
- net N$43: now also IC11A.I, U9.QG; no longer IC1.ENCA_DCIN_CFG5, U1.QB
- net N$44: now also IC16A.I, U9.QE; no longer IC1.SDO_NAO_CFG0, U1.QD
- net N$45: now also IC16A.OE, U9.QF; no longer IC2.OB2, X15-4.S
- net N$46: now also C52.1, IC21.VCC, R39.2; no longer IC2.OA1, X15-2.S
- net N$49: now also C33.2, IC18.CPO; no longer IC2.SDI_NAI_CFG1, IC9A.O
- net N$5: now also C48.1, IC20.AIN_IREF, R36.1; no longer IC4A.I, U1.QG
- net N$50: now also IC18.BRB, R49.2; no longer IC5.OA1, X16-2.S
- net N$51: now also IC18.BRA, R48.2; no longer C37.2, IC5.5VOUT, R70.1
- net N$52: now also C36.1, IC18.AIN_IREF, R28.1; no longer C38.1, IC5.VCP
- net N$53: now also C33.1, IC18.CPI; no longer IC2.SDO_NAO_CFG0, U2.QD
- net N$54: now also IC13A.O, IC18.SCK_CFG2; no longer IC11A.O, IC5.SDI_NAI_CFG1
- net N$57: now also C35.2, IC18.5VOUT, R27.1; no longer IC5.ENCB_DCEN_CFG4, U3.QC
- net N$58: now also C64.1, IC18.VCP; no longer IC5.ENCA_DCIN_CFG5, U3.QB
- net N$59: now also IC18.SDI_NAI_CFG1, IC8A.O; no longer IC11A.OE, U3.QH
- net N$6: now also C45.1, IC20.CPI; no longer IC1.ENCB_DCEN_CFG4, U1.QC
- net N$60: now also C15.1, U4.SS; no longer C49.1, U6.SS
- net N$61: now also IC18.SDO_NAO_CFG0, U6.QD; no longer IC11A.I, U3.QG
- net N$62: now also IC18.ENCB_DCEN_CFG4, U6.QC; no longer IC10A.OE, U3.QF
- net N$63: now also IC18.ENCA_DCIN_CFG5, U6.QB; no longer IC10A.I, U3.QE
- net N$64: now also C3.1, D1.A, Q1.D, R8.1, X11-2.1; no longer C57.1, D3.A, Q2.D, R57.1, X21-2.1
- net N$65: now also IC8A.OE, U6.QH; no longer IC2.ENCA_DCIN_CFG5, U2.QB
- net N$66: now also IC8A.I, U6.QG; no longer IC9A.OE, U2.QH
- net N$67: now also IC13A.I, U6.QE; no longer IC9A.I, U2.QG
- net N$68: now also IC13A.OE, U6.QF; no longer IC8A.OE, U2.QF
- net N$69: now also C34.1, IC18.VCC, R27.2; no longer IC8A.I, U2.QE
- net N$72: now also C39.2, IC19.CPO; no longer IC12.BRA, R30.2
- net N$73: now also C16.1, U4.BOOT; no longer C50.1, U6.BOOT
- net N$74: now also IC19.BRB, R51.2; no longer C62.1, IC12.AIN_IREF, R35.1
- net N$75: now also IC19.BRA, R50.2; no longer C39.1, IC12.CPI
- net N$76: now also C42.1, IC19.AIN_IREF, R32.1; no longer IC12.SCK_CFG2, IC13A.O
- net N$79: now also C39.1, IC19.CPI; no longer C65.2, IC12.5VOUT, R71.1
- net N$8: now also LED7.C, R64.2; no longer LED8.C, R45.2
- net N$80: now also IC14A.O, IC19.SCK_CFG2; no longer C66.1, IC12.VCP
- net N$81: now also IC19.OB2, J503-4.S; no longer IC12.SDI_NAI_CFG1, IC14A.O
- net N$82: now also IC19.OA1, J503-2.S; no longer IC12.SDO_NAO_CFG0, U4.QD
- net N$83: now also C41.2, IC19.5VOUT, R31.1; no longer IC12.ENCB_DCEN_CFG4, U4.QC
- net N$84: now also C66.1, IC19.VCP; no longer IC12.ENCA_DCIN_CFG5, U4.QB
- net N$85: now also IC19.SDI_NAI_CFG1, IC9A.O; no longer IC14A.OE, U4.QH
- net N$86: now also IC19.SDO_NAO_CFG0, U7.QD; no longer IC14A.I, U4.QG
- net N$87: now also IC19.ENCB_DCEN_CFG4, U7.QC; no longer IC13A.OE, U4.QF
- net N$88: now also C14.1, U4.COMP; no longer C51.1, U6.COMP
- net N$89: now also IC19.ENCA_DCIN_CFG5, U7.QB; no longer C36.1, IC15.AIN_IREF, R50.1
- net N$90: now also IC9A.OE, U7.QH; no longer C9.1, IC15.CPI
- net N$91: now also IC9A.I, U7.QG; no longer IC15.SCK_CFG2, IC16A.O
- net N$92: now also IC14A.I, U7.QE; no longer IC15.OB2, X18-4.S
- net N$93: now also IC14A.OE, U7.QF; no longer IC13A.I, U4.QE
- net N$94: now also C40.1, IC19.VCC, R31.2; no longer IC15.OA1, X18-2.S
- net N$95: now also IC19.OA2, J503-1.S; no longer C68.2, IC15.5VOUT, R52.1
- net N$96: now also LED2.A, R24.1; no longer LED4.A, R11.1
- net N$97: now also C14.2, R20.1; no longer C51.2, R26.1
- net N$98: now also IC19.OB1, J503-3.S; no longer C69.1, IC15.VCP
- net N$99: now also C57.2, IC22.CPO; no longer IC15.SDI_NAI_CFG1, IC17A.O
- net SERVO_0: now also IC2A.I; no longer IC6A.I
- net SERVO_0_EN: now also IC2A.OE, U7.QA; no longer IC6A.OE, U2.QA
- net SERVO_1: now also IC1A.I; no longer IC7A.I
- net SERVO_1_EN: now also IC1A.OE, U8.QA; no longer IC7A.OE, U3.QA
- net SER_2: now also U6.QH_2, U7.SER; no longer U1.QH_2, U2.SER
- net SER_3: now also U7.QH_2, U8.SER; no longer U2.QH_2, U3.SER
- net SER_4: now also U8.QH_2, U9.SER; no longer U3.QH_2, U4.SER
- net SER_5: now also U10.SER, U9.QH_2; no longer U4.QH_2, U5.SER
- net SPI1_CS1: now also U10.RCLK, U6.RCLK, U7.RCLK, U8.RCLK, U9.RCLK; no longer U1.RCLK, U2.RCLK, U3.RCLK, U4.RCLK, U5.RCLK
- net SPI1_MOSI: now also U6.SER; no longer U1.SER
- net SPI1_SCLK: now also U10.SRCLK, U6.SRCLK, U7.SRCLK, U8.SRCLK, U9.SRCLK; no longer U1.SRCLK, U2.SRCLK, U3.SRCLK, U4.SRCLK, U5.SRCLK
- net STEP_E: now also IC21.REFL_STEP; no longer IC12.REFL_STEP
- net STEP_H: now also IC22.REFL_STEP; no longer IC15.REFL_STEP
- net STEP_X: now also IC18.REFL_STEP; no longer IC1.REFL_STEP
- net STEP_Y: now also IC19.REFL_STEP; no longer IC2.REFL_STEP
- net STEP_Z: now also IC20.REFL_STEP; no longer IC5.REFL_STEP
- net SYS_5V: now also C18.1, U1.A0, U1.A1, U1.A2, U1.A3, U1.A4, U1.A5, U1.VDD; no longer C17.1, U11.A0, U11.A1, U11.A2, U11.A3, U11.A4, U11.A5, U11.VDD
- net TERM_EXT1: now also C4.1, R10.2; no longer C26.1, R38.2
- net TERM_EXT2: now also C6.1, R14.2; no longer C46.1, R40.2
- net TERM_HBP: now also C5.1, R11.2; no longer C45.1, R39.2
- net THERM_EXT1_IN: now also R10.1, R9.1, X2-2.S; no longer R13.1, R38.1, U8.28, X8-2.S
- net TRISTATE_STEPPERS: now also IC3A.OE, IC4A.OE, IC5A.OE, IC6A.OE, IC7A.OE, U10.QA; no longer IC18A.OE, IC19A.OE, IC20A.OE, IC21A.OE, IC22A.OE, U5.QA
- net VDD_12V: now also C1.1, C2.1, L1.P$1, R19.1, R24.2, X10-4.S; no longer C53.1, C81.1, L2.P$1, R11.2, R42.1, U8.12, U8.16, U8.17, X12-4.S
- net VDD_5V: now also C10.1, C12.1, C13.1, C8.1, IC1P.VCC, IC2P.VCC, L2.P$1, R1.2, R17.1, R2.2, R3.2, R4.2, R5.2, R6.2, X5-3.S, X6-3.S, X7-3.S, X8-3.S, X9-3.S; no longer C48.1, C80.1, C82.1, C83.1, IC6P.VCC, IC7P.VCC, L1.P$1, R12.1, R61.2, R62.2, R63.2, R64.2, R65.2, R66.2, X1-3.S, X12-3.S, X13-3.S, X19-3.S, X22-3.S
- net VDD_ADC: now also R12.2, R9.2; no longer R17.2, R18.2
- net VDD_IN: now also C11.1, C65.2, C68.2, C70.2, C71.2, C72.2, C73.2, C74.1, C75.1, C76.1, C77.1, C78.1, C79.+, C80.+, C81.+, C82.+, C83.+, C84.1, C85.1, C86.1, C87.1, C88.1, C9.1, D6.C, IC18.VS, IC18.VSA, IC19.VS, IC19.VSA, IC20.VS, IC20.VSA, IC21.VS, IC21.VSA, IC22.VS, IC22.VSA, R26.2, R58.2, R59.2, R62.2, R63.2, R64.1, R8.2, U4.VIN, U5.VIN, X11-1.1, X12-1.1, X12-2.1, X13-1.1, X15-1.S, X16-1.S; no longer C10.1, C19.1, C20.2, C22.2, C27.1, C28.2, C29.1, C31.1, C32.2, C35.2, C38.2, C4.1, C40.1, C43.1, C47.1, C52.1, C6.1, C8.1, C94.+, C95.+, C96.+, C97.+, C98.+, D2.C, IC1.VS, IC1.VSA, IC12.VS, IC12.VSA, IC15.VS, IC15.VSA, IC2.VS, IC2.VSA, IC5.VS, IC5.VSA, R14.2, R16.2, R19.2, R20.2, R21.2, R45.1, R55.2, R56.2, R57.2, U10.VIN, U6.VIN, U8.36, U8.37, U8.38, U8.39, U8.40, X20-1.1, X20-2.1, X21-1.1, X3-1.1, X5-1.S, X6-1.S
- net VIN: now also LED7.A, X14-3.1, X14-4.1; no longer LED8.A, X2-3.1, X2-4.1
- net X_A1: now also IC18.OA1, J504-2.S; no longer IC1.OA1, U8.8, X4-2.S
- net X_A2: now also IC18.OA2, J504-1.S; no longer IC1.OA2, U8.7, X4-1.S
- net X_B1: now also IC18.OB1, J504-3.S; no longer IC1.OB1, U8.6, X4-3.S
- net X_B2: now also IC18.OB2, J504-4.S; no longer IC1.OB2, U8.5, X4-4.S
Other:
- note removed: "Fan drivers"
